File: ESP-BuildStatus-Light/ESP-BuildStatus-Light-Board.sch (KiCad schematic (older format))
At the start: 57 parts, among them J2 CONN_01X16, SW1 SW_Push, U1 APA102C, U10 APA102C, U11 APA102C, U12 APA102C, U13 APA102C, U14 APA102C, U15 APA102C, U16 APA102C, U17 APA102C, U18 APA102C, U19 APA102C, U2 APA102C, U20 APA102C, U21 APA102C, U22 APA102C, U23 APA102C, U24 APA102C, U25 APA102C, U26 APA102C, U27 APA102C, U28 APA102C, U29 APA102C, U3 APA102C, U30 APA102C, U31 APA102C, U32 APA102C, U33 APA102C, U34 APA102C, U35 APA102C, U36 APA102C, U37 APA102C, U38 APA102C, U39 APA102C, U4 APA102C, U40 APA102C, U41 APA102C, U42 APA102C, U43 APA102C, U44 APA102C, U45 APA102C, U46 APA102C, U47 APA102C, U48 APA102C, U49 APA102C, U5 APA102C, U50 WeMos_mini, U51 74HCT541_PWR, U6 APA102C, U7 APA102C, U8 APA102C, U9 APA102C

Commit message: Modified traces from WeMos to Level Shifter
Parts:
- C1: symbol C -> device:C
- J2: symbol CONN_01X16 -> conn:CONN_01X16
- R1, R2: symbol R -> device:R
- RV1: symbol POT -> device:POT
- SW1: symbol SW_Push -> switches:SW_Push
- U1, U10, U11, U12, U13, U14, U15, U16, U17, U18, U19, U2, U20, U21, U22, U23, U24, U25, U26, U27, U28, U29, U3, U30, U31, U32, U33, U34, U35, U36, U37, U38, U39, U4, U40, U41, U42, U43, U44, U45, U46, U47, U48, U49, U5, U6, U7, U8, U9: symbol APA102C -> display:APA102C
- U50: footprint wemos_d1_mini:D1_mini_board -> wemos_d1_mini:D1_mini_board_smd; symbol WeMos_mini -> wemos_mini:WeMos_mini
- U51: symbol 74HCT541_PWR -> 74xx1:74HCT541_PWR
Connections:
- net at U1.1 (D_In), U15.1 (D_In), U22.1 (D_In)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: no longer U1.2 (C_In), U15.2 (C_In), U22.2 (C_In), U29.2 (C_In), U36.2 (C_In), U43.2 (C_In), U50.14 (D7), U8.2 (C_In)
- new net: U1.2 (C_In), U15.2 (C_In), U22.2 (C_In), U29.2 (C_In), U36.2 (C_In), U43.2 (C_In), U50.14 (D7), U8.2 (C_In)

Commit message: fixed problems with circuit and board design
Parts:
- added R3: 1K, Resistors_SMD:R_0603_HandSoldering, symbol device:R
- RV1: value POT -> 5K POT
Connections:
- net +5V: now also R3.1; no longer J2.15 (P15)
- net at U51.13 (Y5): now also J2.14 (P14); no longer J2.10 (P10)
- net at U51.14 (Y4): now also J2.13 (P13); no longer J2.9 (P9)
- net at U51.15 (Y3): now also J2.12 (P12); no longer J2.8 (P8)
- net at U51.16 (Y2): now also J2.11 (P11); no longer J2.7 (P7)
- net at U1.1 (D_In), U15.1 (D_In), U22.1 (D_In)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: now also U50.14 (D7); no longer U50.12 (D5)
- net at U1.2 (C_In), U15.2 (C_In), U22.2 (C_In)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: now also U50.12 (D5); no longer U50.14 (D7)
- new net: J2.15 (P15), R3.2
Changed lines of the file:
@@
 P 5650 3800
 F 0 "RV1" V 5475 3800 50  0000 C CNN
-F 1 "POT" V 5550 3800 50  0000 C CNN
+F 1 "5K POT" V 5550 3800 50  0000 C CNN
 F 2 "Potentiometers:Potentiometer_Triwood_RM-065" H 5650 3800 50  0001 C CNN
 F 3 "" H 5650 3800 50  0001 C CNN
@@
 	6850 4000 6850 3650
 Wire Wire Line
-	6850 3650 6950 3650
-Wire Wire Line
-	6950 3650 6950 3150
-Wire Wire Line
-	7050 3150 7050 3700
-Wire Wire Line
-	7050 3700 6950 3700
-Wire Wire Line
 	6950 3700 6950 4000
 Wire Wire Line
 	7050 4000 7050 3750
 Wire Wire Line
-	7050 3750 7150 3750
-Wire Wire Line
-	7150 3750 7150 3150
-Wire Wire Line
-	7250 3150 7250 3800
-Wire Wire Line
-	7250 3800 7150 3800
-Wire Wire Line
 	7150 3800 7150 4000
 Wire Wire Line
 	7850 3150 7850 3300
 Wire Wire Line
-	7750 3150 7750 3650
-Wire Wire Line
 	7750 3650 8050 3650
-Wire Wire Line
-	8050 3650 8050 3050
 Wire Wire Line
 	7350 5550 7350 5400
@@
 Wire Wire Line
 	6550 3150 6550 3800
-Wire Wire Line
-	5700 5700 5400 5700
-Wire Wire Line
-	5700 4950 5700 5700
-Wire Wire Line
-	5800 5900 5400 5900
-Wire Wire Line
-	5800 5050 5800 5900
 Wire Wire Line
 	2800 7650 2950 7650
@@
 	1550 7950 1550 8650
 Wire Wire Line
-	5700 4950 1350 4950
-Wire Wire Line
-	1350 4950 1350 7750
-Wire Wire Line
 	1450 7650 1450 5050
-Wire Wire Line
-	1450 5050 5800 5050
 Connection ~ 1550 10750
 Connection ~ 1450 8050
@@
 Wire Wire Line
 	1750 10450 1750 11150
+$Comp
+L device:R R3
+U 1 1 5E3FCF83
+P 8050 3400
+F 0 "R3" V 8130 3400 50  0000 C CNN
+F 1 "1K" V 8050 3400 50  0000 C CNN
+F 2 "Resistors_SMD:R_0603_HandSoldering" V 7980 3400 50  0001 C CNN
+F 3 "" H 8050 3400 50  0001 C CNN
+	1    8050 3400
+	1    0    0    -1
+$EndComp
+Wire Wire Line
+	7750 3650 7750 3150
+Wire Wire Line
+	8050 3550 8050 3650
+Wire Wire Line
+	8050 3050 8050 3250
+Wire Wire Line
+	1350 4950 1350 7750
+Wire Wire Line
+	1450 5050 5500 5050
+Wire Wire Line
+	5500 5050 5500 5700
+Wire Wire Line
+	5500 5700 5400 5700
+Wire Wire Line
+	5400 5900 5550 5900
+Wire Wire Line
+	5550 5900 5550 4950
+Wire Wire Line
+	5550 4950 1350 4950
+Text GLabel 6350 2800 1    50   Input ~ 0
+VSS
+Text GLabel 6450 2800 1    50   Input ~ 0
+VDD
+Text GLabel 6550 2800 1    50   Input ~ 0
+V0
+Text GLabel 6650 2800 1    50   Input ~ 0
+RS
+Text GLabel 6750 2800 1    50   Input ~ 0
+RW
+Text GLabel 6850 2800 1    50   Input ~ 0
+E
+Text GLabel 6950 2800 1    50   Input ~ 0
+D0
+Text GLabel 7050 2800 1    50   Input ~ 0
+D1
+Text GLabel 7150 2800 1    50   Input ~ 0
+D2
+Text GLabel 7250 2800 1    50   Input ~ 0
+D3
+Text GLabel 7350 2800 1    50   Input ~ 0
+D4
+Text GLabel 7450 2800 1    50   Input ~ 0
+D5
+Text GLabel 7550 2800 1    50   Input ~ 0
+D6
+Text GLabel 7650 2800 1    50   Input ~ 0
+D7
+Text GLabel 7750 2800 1    50   Input ~ 0
+A
+Text GLabel 7850 2800 1    50   Input ~ 0
+K
+Wire Wire Line
+	7650 3800 7650 3150
+Wire Wire Line
+	7150 3800 7650 3800
+Wire Wire Line
+	7550 3750 7550 3150
+Wire Wire Line
+	7050 3750 7550 3750
+Wire Wire Line
+	7450 3700 7450 3150
+Wire Wire Line
+	6950 3700 7450 3700
+Wire Wire Line
+	7350 3650 7350 3150
+Wire Wire Line
+	6850 3650 7350 3650
 $EndSCHEMATC
