File: ESP-BuildStatus-Light/_autosave-ESP-BuildStatus-Light-Board.kicad_pcb (KiCad board)
At the start: 2 copper layers, 113 x 126.6 mm, 64 parts, among them J2 CONN_01X16, SW1 SW_Push, U1 APA102C, U10 APA102C, U11 APA102C, U12 APA102C, U13 APA102C, U14 APA102C, U15 APA102C, U16 APA102C, U17 APA102C, U18 APA102C, U19 APA102C, U2 APA102C, U20 APA102C, U21 APA102C, U22 APA102C, U23 APA102C, U24 APA102C, U25 APA102C, U26 APA102C, U27 APA102C, U28 APA102C, U29 APA102C, U3 APA102C, U30 APA102C, U31 APA102C, U32 APA102C, U33 APA102C, U34 APA102C, U35 APA102C, U36 APA102C, U37 APA102C, U38 APA102C, U39 APA102C, U4 APA102C, U40 APA102C, U41 APA102C, U42 APA102C, U43 APA102C, U44 APA102C, U45 APA102C, U46 APA102C, U47 APA102C, U48 APA102C, U49 APA102C, U5 APA102C, U50 WeMos_mini, U51 74HCT541_PWR, U6 APA102C, U7 APA102C, U8 APA102C, U9 APA102C

Commit message: fixed problems with circuit and board design
Parts:
- RV1: value POT -> 5K POT
Connections:
- U50 pad 12: Net-(U1-Pad1) -> Net-(U1-Pad2)
- U50 pad 14: Net-(U1-Pad2) -> Net-(U1-Pad1)
- U51 pad 13: Net-(J2-Pad10) -> Net-(J2-Pad14)
- U51 pad 14: Net-(J2-Pad9) -> Net-(J2-Pad13)
- U51 pad 15: Net-(J2-Pad8) -> Net-(J2-Pad12)
- U51 pad 16: Net-(J2-Pad7) -> Net-(J2-Pad11)
Routing:
- net Net-(J2-Pad14): track 0.00 -> 24.9 mm
- net Net-(J2-Pad13): track 0.00 -> 22.0 mm
- net Net-(J2-Pad12): track 0.00 -> 19.2 mm
- net Net-(J2-Pad11): track 0.00 -> 16.4 mm
- net Net-(J2-Pad10): track 14.8 -> 0.00 mm
- net Net-(J2-Pad9): track 12.0 -> 0.00 mm
- net Net-(J2-Pad8): track 9.95 -> 0.00 mm
- net Net-(J2-Pad7): track 8.52 -> 0.00 mm
- net Net-(U1-Pad1): track 187.4 -> 193.7 mm
- net Net-(U1-Pad2): track 176.6 -> 173.8 mm
- net GND: track 120.8 -> 121.9 mm
